Commit message: path correction

File: urdf/hole_plan.urdf (robot description, URDF)
Before this commit: robot hole, 1 links, 0 joints
Links:
- link base_link: geometry visual mesh filename=meshes/rectangular_hole.obj

File: urdf/hole_uncertain.urdf (robot description, URDF)
Before this commit: robot hole, 1 links, 0 joints
Links:
- link base_link: geometry visual mesh filename=meshes/hole_uncertain.obj
