Commit message: changes relative path

File: urdf/panda_fr3.urdf (robot description, URDF)
Before this commit: robot panda, 11 links, 10 joints
Links:
- link panda_hand: geometry collision mesh filename=./meshes/hand_simple.obj; visual mesh filename=./meshes/hand.obj
- link panda_leftfinger: geometry collision mesh filename=./meshes/finger_simple.obj; visual mesh filename=./meshes/finger.obj
- link panda_link0: geometry collision mesh filename=./meshes/link0_simple.obj; visual mesh filename=./meshes/link0.obj
- link panda_link1: geometry collision mesh filename=./meshes/link1_simple.obj; visual mesh filename=./meshes/link1.obj
- link panda_link2: geometry collision mesh filename=./meshes/link2_simple.obj; visual mesh filename=./meshes/link2.obj
- link panda_link3: geometry collision mesh filename=./meshes/link3_simple.obj; visual mesh filename=./meshes/link3.obj
- link panda_link4: geometry collision mesh filename=./meshes/link4_simple.obj; visual mesh filename=./meshes/link4.obj
- link panda_link5: geometry collision mesh filename=./meshes/link5_simple.obj; visual mesh filename=./meshes/link5.obj
- link panda_link6: geometry collision mesh filename=./meshes/link6_simple.obj; visual mesh filename=./meshes/link6.obj
- link panda_link7: geometry collision mesh filename=./meshes/link7_simple.obj; visual mesh filename=./meshes/link7.obj
- link panda_rightfinger: geometry collision mesh filename=./meshes/finger_simple.obj; visual mesh filename=./meshes/finger.obj
